Commit message: Publish YAW paper code and result data

File: assets/robots/yaw_bot/yaw_bot.urdf (robot description, URDF)
Before this commit: robot yaw_bot, 7 links, 6 joints
Joints:
- joint L_leg1_r_4: limit lower=0.174533 upper=1.48353 effort=100 velocity=20 -> effort=100 velocity=20; type revolute -> continuous
- joint R_leg1_r_9: limit lower=-1.48353 upper=-0.174533 effort=100 velocity=20 -> effort=100 velocity=20; type revolute -> continuous
